Commit message: feat(aha_description): wheel_radius 0.075 -> 0.042 from CAD
Extracted from upstream/Astra_Hardwares/Astra/Astra.STEP:
the HB-139 drive-wheel subassembly has exactly 4 CYLINDRICAL_SURFACE
entities at r=42.00mm (left+right x outer+inner), so drive wheel
diameter is 84mm — much smaller than the 150mm we'd assumed.

Also update controllers.yaml diff_drive_controller.wheel_radius so
odometry matches physical rolling distance.

Cannot yet extract wheel_separation or AuxWheel (caster) size from the
STEP without walking the assembly transform hierarchy — regex on
CARTESIAN_POINTs only gives local-part coords. Documented in
docs/cad-measurements.md how to do it with FreeCAD when available.

Co-Authored-By: Claude Opus 4.7 <noreply@anthropic.com>

File: overlay_ws/src/aha_description/urdf/mobile_base.xacro (robot description, xacro)
@@ -2,9 +2,13 @@
 <!--
   Differential-drive base added under the existing base_link mesh.
-  Provisional dimensions (base is 550x500 mm / ~51 kg per the AhaRobot paper);
-  refine once real chassis / wheel specs are confirmed:
-    wheel_radius     = 0.075 m
-    wheel_separation = 0.40  m
-    caster_radius    = 0.03  m
+  Dimensions:
+    wheel_radius     = 0.042 m  (MEASURED from upstream/Astra_Hardwares/Astra/Astra.STEP:
+                                  the HB-139 drive-wheel subassembly has 4
+                                  CYLINDRICAL_SURFACE entities at r=42.00 mm.
+                                  See docs/cad-measurements.md)
+    wheel_separation = 0.40  m  (ESTIMATED from paper "base 550x500 mm";
+                                  needs FreeCAD/CAD viewer to confirm from
+                                  Astra.STEP assembly transforms.)
+    caster_radius    = 0.03  m  (ESTIMATED; AuxWheel geometry not yet extracted.)
   Frames:
     base_footprint   — flat frame on the ground plane (Nav2 default root)
@@ -15,5 +19,5 @@
 -->
 <robot xmlns:xacro="http://www.ros.org/wiki/xacro">
-  <xacro:property name="wheel_radius"     value="0.075"/>
+  <xacro:property name="wheel_radius"     value="0.042"/>
   <xacro:property name="wheel_width"      value="0.04"/>
   <xacro:property name="wheel_separation" value="0.40"/>
