Commit message: Refactor documents

File: overlay_ws/src/aha_description/urdf/mobile_base.xacro (robot description, xacro)
@@ -6,5 +6,5 @@
                                   the HB-139 drive-wheel subassembly has 4
                                   CYLINDRICAL_SURFACE entities at r=42.00 mm.
-                                  See docs/cad-measurements.md)
+                                  See docs/context/cad.md)
     wheel_separation = 0.40  m  (ESTIMATED from paper "base 550x500 mm";
                                   needs FreeCAD/CAD viewer to confirm from

File: overlay_ws/src/aha_description/urdf/ros2_control.xacro (robot description, xacro)
@@ -2,9 +2,8 @@
 <!--
   ros2_control block for AhaRobot.
-  Design note:
-    Upstream joint <limit> tags are all effort=0 velocity=0. We do NOT patch
-    those in the URDF (would require rewriting the upstream file). Instead we
-    enforce real limits at the controller layer via config/joint_limits.yaml
-    (loaded by joint_limits_interface).
+  Joint limits:
+    Upstream joint <limit> tags are all effort=0 velocity=0. At build time,
+    scripts/patch_limits.py writes urdf/astra_description_patched.urdf into
+    the install tree. aha_robot.urdf.xacro includes that generated copy.
   Joints exposed to controllers:
     - drive: left_wheel_joint, right_wheel_joint         (velocity)
