Commit message: fix(bringup): Japan Open会場で起動直後に昇降が下限の外に残る問題を直す
Japan Open会場（生成時の高さ0.10 m）では、着地の衝撃で昇降が一時的に
5 mm以上沈む。0.005 mの余裕では物理限界に触れて張り付き、
限界に触れない場合も、lift_controllerが沈んだ位置（約-0.005 m）を保持していた。
URDFの下限0 mより下なので、開始状態を指定しないMoveItの計画が拒否される。

- 物理限界の余裕を0.05（m / rad）に広げる
- 昇降の位置指令の初期値を0 mにする（ros2_controlのinitial_value）。
  lift_controllerは起動時にこの指令値を保持するため、昇降は0 mへ戻る。

Refs #31

Co-Authored-By: Claude Opus 5.5 <noreply@anthropic.com>

File: overlay_ws/src/aha_description/urdf/ros2_control.xacro (robot description, xacro)
@@ -17,8 +17,15 @@
 -->
 <robot xmlns:xacro="http://www.ros.org/wiki/xacro">
-  <xacro:macro name="pos_joint" params="name">
+  <xacro:macro name="pos_joint" params="name initial:=''">
     <joint name="${name}">
       <command_interface name="position"/>
-      <state_interface name="position"/>
+      <xacro:if value="${initial == ''}">
+        <state_interface name="position"/>
+      </xacro:if>
+      <xacro:unless value="${initial == ''}">
+        <state_interface name="position">
+          <param name="initial_value">${initial}</param>
+        </state_interface>
+      </xacro:unless>
       <state_interface name="velocity"/>
       <state_interface name="effort"/>
@@ -47,7 +54,10 @@
       <xacro:vel_joint name="left_wheel_joint"/>
       <xacro:vel_joint name="right_wheel_joint"/>
-      <!-- Lift (left + right; treated as 2 DoF for now) -->
-      <xacro:pos_joint name="joint_l1"/>
-      <xacro:pos_joint name="joint_r1"/>
+      <!-- Lift (left + right; treated as 2 DoF for now).
+           initial_value makes gz_ros2_control start the position command at
+           0 m, which lift_controller holds on activation, so the lifts rise
+           back to 0 m after dipping when the robot lands at the spawn. -->
+      <xacro:pos_joint name="joint_l1" initial="0.0"/>
+      <xacro:pos_joint name="joint_r1" initial="0.0"/>
       <!-- Left arm -->
       <xacro:pos_joint name="joint_l2"/>

Commit message: fix(bringup): 昇降の沈み込みを保持力で防ぎ、限界の余裕を小さくする
レビュー指摘への対応。
- 昇降の沈み込みは着地の衝撃（約3 kN）がURDFの力の上限（400 N）を超えるために起きる。
  Gazebo用モデルだけ昇降の力の上限を10 kNにし、摩擦とinitial_valueをやめた。
  起動直後の昇降の最小値は約-1e-10 mになる。
- 沈み込みがなくなったので、物理限界の余裕を全関節0.005（m / rad）に戻した。
  指の可動幅0.06 mに対して0.05は大きく、指が交差・開きすぎる幅を広げていた。
- xacroを1回だけ展開し、robot_state_publisherとGazeboに同じ結果を渡す。
- ros2_control.xacroはmainと同じに戻した（initial_valueが実機設定に入らない）。

Co-Authored-By: Claude Opus 5.5 <noreply@anthropic.com>

File: overlay_ws/src/aha_description/urdf/ros2_control.xacro (robot description, xacro)
@@ -17,15 +17,8 @@
 -->
 <robot xmlns:xacro="http://www.ros.org/wiki/xacro">
-  <xacro:macro name="pos_joint" params="name initial:=''">
+  <xacro:macro name="pos_joint" params="name">
     <joint name="${name}">
       <command_interface name="position"/>
-      <xacro:if value="${initial == ''}">
-        <state_interface name="position"/>
-      </xacro:if>
-      <xacro:unless value="${initial == ''}">
-        <state_interface name="position">
-          <param name="initial_value">${initial}</param>
-        </state_interface>
-      </xacro:unless>
+      <state_interface name="position"/>
       <state_interface name="velocity"/>
       <state_interface name="effort"/>
@@ -54,10 +47,7 @@
       <xacro:vel_joint name="left_wheel_joint"/>
       <xacro:vel_joint name="right_wheel_joint"/>
-      <!-- Lift (left + right; treated as 2 DoF for now).
-           initial_value makes gz_ros2_control start the position command at
-           0 m, which lift_controller holds on activation, so the lifts rise
-           back to 0 m after dipping when the robot lands at the spawn. -->
-      <xacro:pos_joint name="joint_l1" initial="0.0"/>
-      <xacro:pos_joint name="joint_r1" initial="0.0"/>
+      <!-- Lift (left + right; treated as 2 DoF for now) -->
+      <xacro:pos_joint name="joint_l1"/>
+      <xacro:pos_joint name="joint_r1"/>
       <!-- Left arm -->
       <xacro:pos_joint name="joint_l2"/>
