Commit message: add: cameras in sample tasks

File: overlay_ws/src/aha_description/urdf/aha_robot.urdf.xacro (robot description, xacro)
@@ -9,9 +9,10 @@
       the same joints via controller_manager.
     - Adds <gazebo> plugin block for gz_ros2_control (Gazebo Harmonic).
-    - Adds head camera frames and, in sim, its Gazebo sensor (see sensors.xacro).
+    - Adds head camera frames and optional simulated head/wrist cameras.
     - Adds a sim-only 2D LiDAR when lidar:=true (see lidar.xacro).
   Xacro args:
     sim            (true|false)  — include Gazebo plugin, gz_ros2_control plugin
                                    and Gazebo sensors
+    cameras        (true|false)  — head RGB-D and wrist RGB cameras (default: same as sim)
     lidar          (true|false)  — add the sim-only 2D LiDAR (default: same as sim)
     use_sim_time   (true|false)  — inform robot_state_publisher
@@ -19,4 +20,5 @@
 <robot name="aha_robot" xmlns:xacro="http://www.ros.org/wiki/xacro">
   <xacro:arg name="sim" default="true"/>
+  <xacro:arg name="cameras" default="$(arg sim)"/>
   <xacro:arg name="lidar" default="$(arg sim)"/>
   <xacro:arg name="controllers_yaml" default="$(find aha_description)/config/controllers.yaml"/>
@@ -43,5 +45,5 @@
   <!-- 5. Sensors (head camera frames always; Gazebo sensor in sim) -->
   <xacro:include filename="$(find aha_description)/urdf/sensors.xacro"/>
-  <xacro:aha_sensors sim="$(arg sim)"/>
+  <xacro:aha_sensors sim="$(arg sim)" cameras="$(arg cameras)"/>
   <!-- 6. Sim-only 2D LiDAR (used by aha_navigation SLAM) -->
   <xacro:if value="$(arg lidar)">

File: overlay_ws/src/aha_description/urdf/sensors.xacro (robot description, xacro)
@@ -11,4 +11,5 @@
   Gazebo topics (bridged to ROS by aha_perception/launch/perception.launch.py):
     head_camera/{image,depth_image,camera_info}  rgbd_camera, depth aligned to color
+    {left,right}_wrist_camera/{image,camera_info}  RGB cameras
 -->
 <robot xmlns:xacro="http://www.ros.org/wiki/xacro">
@@ -43,5 +44,48 @@
   <xacro:property name="camera_depth_far"          value="10.0"/>
   <xacro:property name="camera_depth_noise_stddev" value="0.005"/>
-  <xacro:macro name="aha_sensors" params="sim">
+  <!-- Virtual wrist mounts, outside the palm and finger meshes (max x < 0.09 m).
+       Both palms have the same local geometry. Look toward the grasp center
+       near (0.063, 0, 0.195), along +z with a small inward tilt.
+       These visual-only mounts add no collision geometry or payload mass. -->
+  <xacro:macro name="aha_wrist_camera" params="side parent">
+    <link name="${side}_wrist_camera_link">
+      <visual>
+        <geometry><box size="0.02 0.025 0.025"/></geometry>
+        <material name="camera_dark_grey"/>
+      </visual>
+    </link>
+    <joint name="${side}_wrist_camera_joint" type="fixed">
+      <parent link="${parent}"/>
+      <child link="${side}_wrist_camera_link"/>
+      <origin xyz="0.115 0 0.045" rpy="0 -1.904 0"/>
+    </joint>
+    <link name="${side}_wrist_camera_optical_frame"/>
+    <joint name="${side}_wrist_camera_optical_joint" type="fixed">
+      <parent link="${side}_wrist_camera_link"/>
+      <child link="${side}_wrist_camera_optical_frame"/>
+      <origin xyz="0.011 0 0" rpy="${-pi/2} 0 ${-pi/2}"/>
+    </joint>
+    <gazebo reference="${side}_wrist_camera_link">
+      <sensor name="${side}_wrist_camera" type="camera">
+        <pose>0.011 0 0 0 0 0</pose>
+        <always_on>true</always_on>
+        <update_rate>${camera_rate}</update_rate>
+        <visualize>false</visualize>
+        <topic>${side}_wrist_camera/image</topic>
+        <gz_frame_id>${side}_wrist_camera_optical_frame</gz_frame_id>
+        <camera>
+          <camera_info_topic>${side}_wrist_camera/camera_info</camera_info_topic>
+          <horizontal_fov>${pi/2}</horizontal_fov>
+          <image>
+            <width>${camera_width}</width>
+            <height>${camera_height}</height>
+            <format>R8G8B8</format>
+          </image>
+          <clip><near>0.02</near><far>3.0</far></clip>
+        </camera>
+      </sensor>
+    </gazebo>
+  </xacro:macro>
+  <xacro:macro name="aha_sensors" params="sim cameras:=true">
     <link name="camera_link">
       <visual>
@@ -62,4 +106,5 @@
     </joint>
     <xacro:if value="${sim}">
+      <xacro:if value="${cameras}">
       <gazebo reference="camera_link">
         <sensor name="head_camera" type="rgbd_camera">
@@ -96,4 +141,7 @@
         </sensor>
       </gazebo>
+      <xacro:aha_wrist_camera side="left" parent="link_l6"/>
+      <xacro:aha_wrist_camera side="right" parent="link_r6"/>
+      </xacro:if>
     </xacro:if>
   </xacro:macro>

File: overlay_ws/src/aha_sim_tasks/worlds/task_tables.sdf.xacro (robot description, xacro)
@@ -2,4 +2,5 @@
 <sdf version="1.10" xmlns:xacro="http://www.ros.org/wiki/xacro">
   <xacro:arg name="scene_config" default="$(find aha_sim_tasks)/config/scene.json"/>
+  <xacro:arg name="cameras" default="true"/>
   <xacro:property name="scene" value="${xacro.load_yaml('$(arg scene_config)')}"/>
   <world name="task_tables">
@@ -11,4 +12,9 @@
     <plugin filename="gz-sim-user-commands-system" name="gz::sim::systems::UserCommands"/>
     <plugin filename="gz-sim-scene-broadcaster-system" name="gz::sim::systems::SceneBroadcaster"/>
+    <xacro:if value="$(arg cameras)">
+      <plugin filename="gz-sim-sensors-system" name="gz::sim::systems::Sensors">
+        <render_engine>ogre2</render_engine>
+      </plugin>
+    </xacro:if>
     <plugin filename="aha_task_evaluation" name="aha_sim_tasks::EvaluationSystem">
       <robot_model>${scene.entities.robot_model}</robot_model>

Commit message: feat: introduce ycb objects to sim

File: overlay_ws/src/aha_description/urdf/aha_robot.urdf.xacro (robot description, xacro)
@@ -21,4 +21,6 @@
   <xacro:arg name="sim" default="true"/>
   <xacro:arg name="cameras" default="$(arg sim)"/>
+  <xacro:arg name="camera_rgb_noise_stddev" default="0.003"/>
+  <xacro:arg name="initial_lift" default="0.0"/>
   <xacro:arg name="lidar" default="$(arg sim)"/>
   <xacro:arg name="controllers_yaml" default="$(find aha_description)/config/controllers.yaml"/>

File: overlay_ws/src/aha_description/urdf/ros2_control.xacro (robot description, xacro)
@@ -17,8 +17,12 @@
 -->
 <robot xmlns:xacro="http://www.ros.org/wiki/xacro">
-  <xacro:macro name="pos_joint" params="name">
+  <xacro:macro name="pos_joint" params="name initial:=0.0">
     <joint name="${name}">
       <command_interface name="position"/>
-      <state_interface name="position"/>
+      <state_interface name="position">
+        <xacro:if value="${float(initial) > 0.0}">
+          <param name="initial_value">${initial}</param>
+        </xacro:if>
+      </state_interface>
       <state_interface name="velocity"/>
       <state_interface name="effort"/>
@@ -48,6 +52,6 @@
       <xacro:vel_joint name="right_wheel_joint"/>
       <!-- Lift (left + right; treated as 2 DoF for now) -->
-      <xacro:pos_joint name="joint_l1"/>
-      <xacro:pos_joint name="joint_r1"/>
+      <xacro:pos_joint name="joint_l1" initial="$(arg initial_lift)"/>
+      <xacro:pos_joint name="joint_r1" initial="$(arg initial_lift)"/>
       <!-- Left arm -->
       <xacro:pos_joint name="joint_l2"/>

File: overlay_ws/src/aha_description/urdf/sensors.xacro (robot description, xacro)
@@ -40,8 +40,8 @@
   <!-- 69 deg, D435i color HFOV -->
   <xacro:property name="camera_hfov"   value="1.204"/>
-  <!-- Depth range and noise -->
+  <!-- Depth range; benchmark depth noise is applied by aha_sim_tasks to policy observations. -->
   <xacro:property name="camera_depth_near"         value="0.28"/>
   <xacro:property name="camera_depth_far"          value="10.0"/>
-  <xacro:property name="camera_depth_noise_stddev" value="0.005"/>
+  <xacro:property name="camera_rgb_noise_stddev" value="$(arg camera_rgb_noise_stddev)"/>
   <!-- Virtual wrist mounts, outside the palm and finger meshes (max x < 0.09 m).
        Both palms have the same local geometry. Look toward the grasp center
@@ -83,4 +83,5 @@
           </image>
           <clip><near>0.02</near><far>3.0</far></clip>
+          <noise><type>gaussian</type><mean>0.0</mean><stddev>${camera_rgb_noise_stddev}</stddev></noise>
         </camera>
       </sensor>
@@ -136,5 +137,5 @@
               <type>gaussian</type>
               <mean>0.0</mean>
-              <stddev>${camera_depth_noise_stddev}</stddev>
+              <stddev>${camera_rgb_noise_stddev}</stddev>
             </noise>
           </camera>

File: overlay_ws/src/aha_sim_tasks/worlds/task_tables.sdf.xacro (robot description, xacro)
@@ -5,16 +5,41 @@
   <xacro:arg name="ground_truth" default="false"/>
   <xacro:property name="scene" value="${xacro.load_yaml('$(arg scene_config)')}"/>
+  <xacro:macro name="table" params="name position color">
+    <model name="${name}">
+      <static>true</static>
+      <pose>${position[0]} ${position[1]} ${position[2]} 0 0 0</pose>
+      <link name="top">
+        <collision name="collision">
+          <geometry><box><size>${scene.table_size[0]} ${scene.table_size[1]} ${scene.table_size[2]}</size></box></geometry>
+          <surface><friction><ode><mu>${scene.physics.table_friction}</mu><mu2>${scene.physics.table_friction}</mu2></ode></friction></surface>
+        </collision>
+        <visual name="visual">
+          <geometry><box><size>${scene.table_size[0]} ${scene.table_size[1]} ${scene.table_size[2]}</size></box></geometry>
+          <material><ambient>${color} 1</ambient><diffuse>${color} 1</diffuse></material>
+        </visual>
+      </link>
+      <xacro:property name="leg_height" value="${position[2] - scene.table_size[2]/2}"/>
+      <xacro:macro name="leg" params="suffix x y">
+        <link name="leg_${suffix}">
+          <pose>${x} ${y} ${-scene.table_size[2]/2 - leg_height/2} 0 0 0</pose>
+          <collision name="collision"><geometry><box><size>0.04 0.04 ${leg_height}</size></box></geometry></collision>
+          <visual name="visual"><geometry><box><size>0.04 0.04 ${leg_height}</size></box></geometry>
+            <material><ambient>0.18 0.16 0.14 1</ambient><diffuse>0.25 0.22 0.19 1</diffuse></material>
+          </visual>
+        </link>
+      </xacro:macro>
+      <xacro:leg suffix="front_left" x="${-scene.table_size[0]/2 + 0.04}" y="${scene.table_size[1]/2 - 0.04}"/>
+      <xacro:leg suffix="front_right" x="${-scene.table_size[0]/2 + 0.04}" y="${-scene.table_size[1]/2 + 0.04}"/>
+      <xacro:leg suffix="back_left" x="${scene.table_size[0]/2 - 0.04}" y="${scene.table_size[1]/2 - 0.04}"/>
+      <xacro:leg suffix="back_right" x="${scene.table_size[0]/2 - 0.04}" y="${-scene.table_size[1]/2 + 0.04}"/>
+    </model>
+  </xacro:macro>
   <world name="task_tables">
-    <physics name="1ms" type="ignored">
-      <max_step_size>0.001</max_step_size>
-      <real_time_factor>1.0</real_time_factor>
-    </physics>
+    <physics name="1ms" type="ignored"><max_step_size>0.001</max_step_size><real_time_factor>1.0</real_time_factor></physics>
     <plugin filename="gz-sim-physics-system" name="gz::sim::systems::Physics"/>
     <plugin filename="gz-sim-user-commands-system" name="gz::sim::systems::UserCommands"/>
     <plugin filename="gz-sim-scene-broadcaster-system" name="gz::sim::systems::SceneBroadcaster"/>
     <xacro:if value="$(arg cameras)">
-      <plugin filename="gz-sim-sensors-system" name="gz::sim::systems::Sensors">
-        <render_engine>ogre2</render_engine>
-      </plugin>
+      <plugin filename="gz-sim-sensors-system" name="gz::sim::systems::Sensors"><render_engine>ogre2</render_engine></plugin>
     </xacro:if>
     <plugin filename="aha_task_evaluation" name="aha_sim_tasks::EvaluationSystem">
@@ -26,64 +51,19 @@
       <right_finger_link>${scene.entities.right_finger_link}</right_finger_link>
       <left_finger_link>${scene.entities.left_finger_link}</left_finger_link>
+      <destination_model>destination_table</destination_model>
     </plugin>
     <light type="directional" name="sun">
       <pose>0 0 10 0 0 0</pose>
-      <diffuse>0.8 0.8 0.8 1</diffuse>
-      <direction>-0.5 0.1 -0.9</direction>
+      <diffuse>${scene.lighting.intensity} ${scene.lighting.intensity} ${scene.lighting.intensity} 1</diffuse>
+      <direction>${scene.lighting.direction[0]} ${scene.lighting.direction[1]} ${scene.lighting.direction[2]}</direction>
     </light>
-    <model name="ground_plane">
-      <static>true</static>
-      <link name="link">
-        <collision name="collision">
-          <geometry><plane><normal>0 0 1</normal><size>5 5</size></plane></geometry>
-        </collision>
-        <visual name="visual">
-          <geometry><plane><normal>0 0 1</normal><size>5 5</size></plane></geometry>
-          <material><ambient>0.65 0.65 0.65 1</ambient><diffuse>0.75 0.75 0.75 1</diffuse></material>
-        </visual>
-      </link>
-    </model>
-    <model name="source_table">
-      <static>true</static>
-      <pose>${scene.source_position[0]} ${scene.source_position[1]} ${scene.source_position[2] - scene.apple_radius - scene.table_size[2]/2} 0 0 0</pose>
-      <link name="top">
-        <collision name="collision"><geometry><box><size>${scene.table_size[0]} ${scene.table_size[1]} ${scene.table_size[2]}</size></box></geometry></collision>
-        <visual name="visual">
-          <geometry><box><size>${scene.table_size[0]} ${scene.table_size[1]} ${scene.table_size[2]}</size></box></geometry>
-          <material><ambient>0.38 0.22 0.12 1</ambient><diffuse>0.48 0.28 0.16 1</diffuse></material>
-        </visual>
-      </link>
-    </model>
-    <model name="destination_table">
-      <static>true</static>
-      <pose>${scene.destination_position[0]} ${scene.destination_position[1]} ${scene.destination_position[2] - scene.apple_radius - scene.table_size[2]/2} 0 0 0</pose>
-      <link name="top">
-        <collision name="collision"><geometry><box><size>${scene.table_size[0]} ${scene.table_size[1]} ${scene.table_size[2]}</size></box></geometry></collision>
-        <visual name="visual">
-          <geometry><box><size>${scene.table_size[0]} ${scene.table_size[1]} ${scene.table_size[2]}</size></box></geometry>
-          <material><ambient>0.08 0.45 0.12 1</ambient><diffuse>0.10 0.65 0.16 1</diffuse></material>
-        </visual>
-      </link>
-    </model>
-    <model name="${scene.entities.object_model}">
-      <pose>${scene.source_position[0]} ${scene.source_position[1]} ${scene.source_position[2]} 0 0 0</pose>
-      <link name="${scene.entities.object_link}">
-        <inertial>
-          <mass>0.08</mass>
-          <inertia>
-            <ixx>${0.4 * 0.08 * scene.apple_radius**2}</ixx><iyy>${0.4 * 0.08 * scene.apple_radius**2}</iyy><izz>${0.4 * 0.08 * scene.apple_radius**2}</izz>
-            <ixy>0</ixy><ixz>0</ixz><iyz>0</iyz>
-          </inertia>
-        </inertial>
-        <collision name="${scene.entities.object_collision}">
-          <geometry><sphere><radius>${scene.apple_radius}</radius></sphere></geometry>
-          <surface><friction><ode><mu>1.0</mu><mu2>1.0</mu2></ode></friction></surface>
-        </collision>
-        <visual name="fruit_visual">
-          <geometry><sphere><radius>${scene.apple_radius}</radius></sphere></geometry>
-          <material><ambient>0.65 0.03 0.02 1</ambient><diffuse>0.90 0.04 0.02 1</diffuse></material>
-        </visual>
-      </link>
-    </model>
+    <model name="ground_plane"><static>true</static><link name="link">
+      <collision name="collision"><geometry><plane><normal>0 0 1</normal><size>8 8</size></plane></geometry></collision>
+      <visual name="visual"><geometry><plane><normal>0 0 1</normal><size>8 8</size></plane></geometry>
+        <material><ambient>0.65 0.65 0.65 1</ambient><diffuse>0.75 0.75 0.75 1</diffuse></material>
+      </visual>
+    </link></model>
+    <xacro:table name="source_table" position="${scene.source_table_position}" color="0.48 0.28 0.16"/>
+    <xacro:table name="destination_table" position="${scene.destination_table_position}" color="0.10 0.55 0.16"/>
   </world>
 </sdf>
