Commit message: fix(description): sim の頭部カメラの水平画角を実機 D435i のカラー (640x480, fx 602.9) に合わせる

File: overlay_ws/src/aha_description/urdf/sensors.xacro (robot description, xacro)
@@ -38,6 +38,8 @@
   <xacro:property name="camera_height" value="480"/>
   <xacro:property name="camera_rate"   value="15"/>
-  <!-- 69 deg, D435i color HFOV -->
-  <xacro:property name="camera_hfov"   value="1.204"/>
+  <!-- 55.9 deg: fx 602.9 px at 640x480, the real D435i color CameraInfo
+       (tools/perception/plane_bench/real_frames, 2026-10-04). The 69 deg
+       datasheet HFOV is for 16:9; 640x480 crops the sides. -->
+  <xacro:property name="camera_hfov"   value="0.9759"/>
   <!-- Depth range; benchmark depth noise is applied by aha_sim_tasks to policy observations. -->
   <xacro:property name="camera_depth_near"         value="0.28"/>

Commit message: feat: introduce ycb objects

File: overlay_ws/src/aha_description/urdf/sensors.xacro (robot description, xacro)
@@ -44,19 +44,22 @@
   <xacro:property name="camera_depth_far"          value="10.0"/>
   <xacro:property name="camera_rgb_noise_stddev" value="$(arg camera_rgb_noise_stddev)"/>
-  <!-- Virtual wrist mounts, outside the palm and finger meshes (max x < 0.09 m).
-       Both palms have the same local geometry. Look toward the grasp center
-       near (0.063, 0, 0.195), along +z with a small inward tilt.
-       These visual-only mounts add no collision geometry or payload mass. -->
+  <!-- The Camera component (including its bracket) is already part of both
+       upstream link_[lr]6.STL meshes. Use its CAD placement from
+       Astra_Hardwares/Astra/Astra.STEP instead of adding another camera body.
+       CAD link6 coordinates (X,Y,Z) map to wrist (60-Y, X, 28+Z), in mm.
+       The Camera origin is (0,34,73) mm, and its lens looks 30 degrees down
+       from wrist +z. Wrist +x points DOWN with the arm extended, so this
+       placement is above the grasp center (0.063, 0, 0.195).
+       The lens front is 16 mm along the camera's viewing axis. These are CAD
+       design values; optical calibration on the real robot is not available. -->
+  <xacro:property name="wrist_camera_mount_xyz" value="0.026 0 0.101"/>
+  <xacro:property name="wrist_camera_mount_pitch" value="${-pi/3}"/>
+  <xacro:property name="wrist_camera_lens_offset" value="0.016"/>
   <xacro:macro name="aha_wrist_camera" params="side parent">
-    <link name="${side}_wrist_camera_link">
-      <visual>
-        <geometry><box size="0.02 0.025 0.025"/></geometry>
-        <material name="camera_dark_grey"/>
-      </visual>
-    </link>
+    <link name="${side}_wrist_camera_link"/>
     <joint name="${side}_wrist_camera_joint" type="fixed">
       <parent link="${parent}"/>
       <child link="${side}_wrist_camera_link"/>
-      <origin xyz="0.115 0 0.045" rpy="0 -1.904 0"/>
+      <origin xyz="${wrist_camera_mount_xyz}" rpy="0 ${wrist_camera_mount_pitch} 0"/>
     </joint>
     <link name="${side}_wrist_camera_optical_frame"/>
@@ -64,9 +67,9 @@
       <parent link="${side}_wrist_camera_link"/>
       <child link="${side}_wrist_camera_optical_frame"/>
-      <origin xyz="0.011 0 0" rpy="${-pi/2} 0 ${-pi/2}"/>
+      <origin xyz="${wrist_camera_lens_offset} 0 0" rpy="${-pi/2} 0 ${-pi/2}"/>
     </joint>
     <gazebo reference="${side}_wrist_camera_link">
       <sensor name="${side}_wrist_camera" type="camera">
-        <pose>0.011 0 0 0 0 0</pose>
+        <pose>${wrist_camera_lens_offset} 0 0 0 0 0</pose>
         <always_on>true</always_on>
         <update_rate>${camera_rate}</update_rate>
